File: kicad/video_rider_st.kicad_sch (KiCad schematic)
At the start: 2 parts

Commit message: Most basic components now on schematic.
Parts:
- added C1, C2: 1u, symbol Device:C
- added C3, C4, C5, C6, C7: 100n, symbol Device:C
- added D1: D_Schottky, symbol Device:D_Schottky
- added J1, J3, J6, J7: Conn_01x20, symbol Connector_Generic:Conn_01x20
- added J2: Conn_01x16_Female, symbol Connector:Conn_01x16_Female
- added J4: Conn_01x02_Male, symbol Connector:Conn_01x02_Male
- added J5: Conn_01x03_Male, symbol Connector:Conn_01x03_Male
- added R1: 10k, symbol Device:R
- added R2, R3, R4: 6k8, symbol Device:R
- added U10: ST_GLUE_PHY, Package_LCC:PLCC-68_THT-Socket, symbol st_glue:ST_GLUE_PHY
- added U11: ST_GLUE_SOCKET, Package_LCC:PLCC-68_THT-Socket, symbol st_glue:ST_GLUE_SOCKET
- added U3: Pico, RPi_Pico:RPi_Pico_SMD_TH, symbol MCU_RaspberryPi_and_Boards:Pico
- added U4, U5, U6, U7: 74HC245, symbol 74xx:74HC245
- added U8: LM1117-3.3, symbol Regulator_Linear:LM1117-3.3
- added U9: XC95144XL-TQ100, Package_QFP:TQFP-100_14x14mm_P0.5mm, symbol CPLD_Xilinx:XC95144XL-TQ100
- added X1: CXO_DIP14, Oscillator:Oscillator_DIP-14, symbol Oscillator:CXO_DIP14
- gave numbers to parts that had none: 2
Connections:
- net 5V: now also C1.1, C4.1, D1.2 (A), R1.1, U10.1 (VCC), U11.1 (VCC), U4.20 (VCC), U5.20 (VCC), U6.20 (VCC), U7.20 (VCC), U8.3 (VI), X1.14 (Vcc)
- net A1: now also U10.56 (A1), U11.56 (A1), U9.53 (P53)
- net A2: now also U10.57 (A2), U11.57 (A2), U9.52 (P52)
- net A3: now also U10.58 (A3), U11.58 (A3), U9.50 (P50)
- net A4: now also U10.59 (A4), U11.59 (A4), U9.86 (P86)
- net A5: now also U10.60 (A5), U11.60 (A5), U9.85 (P85)
- net B0: now also U4.5 (A3)
- net B1: now also U4.6 (A4)
- net B2: now also U4.7 (A5)
- net B_OUT0: now also U4.15 (B3), U6.13 (B5)
- net B_OUT1: now also U4.14 (B4), U6.12 (B6)
- net B_OUT2: now also U4.13 (B5), U6.11 (B7)
- net D0: now also J3.3 (Pin_3), U10.48 (D0), U11.48 (D0)
- net D1: now also J3.4 (Pin_4), U10.49 (D1), U11.49 (D1)
- net D10: now also J3.13 (Pin_13)
- net D11: now also J3.14 (Pin_14)
- net D12: now also J3.15 (Pin_15)
- net D13: now also J3.16 (Pin_16)
- net D14: now also J3.17 (Pin_17)
- net D15: now also J3.18 (Pin_18)
- net D2: now also J3.5 (Pin_5)
- net D3: now also J3.6 (Pin_6)
- net D4: now also J3.7 (Pin_7)
- net D5: now also J3.8 (Pin_8)
- net D6: now also J3.9 (Pin_9)
- net D7: now also J3.10 (Pin_10)
- net D8: now also J3.11 (Pin_11)
- net D9: now also J3.12 (Pin_12)
- net DE: now also U10.39 (DE), U11.39 (DE)
- net G0: now also U4.2 (A0)
- net G1: now also U4.3 (A1)
- net G2: now also U4.4 (A2)
- net GND: now also C1.2, C2.2, C3.2, C4.2, C5.2, C6.2, C7.2, J1.1 (Pin_1), J1.19 (Pin_19), J1.2 (Pin_2), J1.20 (Pin_20), J2.1 (Pin_1), J2.16 (Pin_16), J3.1 (Pin_1), J3.19 (Pin_19), J3.2 (Pin_2), J3.20 (Pin_20), J4.2 (Pin_2), J6.1 (Pin_1), J6.19 (Pin_19), J6.2 (Pin_2), J6.20 (Pin_20), J7.1 (Pin_1), J7.19 (Pin_19), J7.2 (Pin_2), J7.20 (Pin_20), U10.35 (GND), U11.35 (GND), U3.13 (GND), U3.18 (GND), U3.23 (GND), U3.28 (GND), U3.3 (GND), U3.33 (AGND), U3.38 (GND), U3.8 (GND), U4.10 (GND), U5.10 (GND), U6.10 (GND), U7.10 (GND), U8.1 (GND), U9.100 (GND), U9.21 (GND), U9.31 (GND), U9.44 (GND), U9.62 (GND), U9.69 (GND), U9.75 (GND), U9.84 (GND), X1.7 (GND)
- net G_OUT0: now also U4.18 (B0), U6.17 (B1)
- net G_OUT1: now also U4.17 (B1), U6.16 (B2)
- net G_OUT2: now also U4.16 (B2), U6.15 (B3)
- net MONO: now also U5.5 (A3)
- net MONO_OUT: now also U5.15 (B3)
- net R0: now also U5.2 (A0)
- net R1: now also U5.3 (A1)
- net R2: now also U5.4 (A2)
- net RW: now also U10.55 (R/~{W}), U11.55 (R/~{W}), U9.11 (P11)
- net R_OUT0: now also U5.18 (B0), U7.17 (B1)
- net R_OUT1: now also U5.17 (B1), U7.16 (B2)
- net R_OUT2: now also U5.16 (B2), U7.15 (B3)
- new net: J4.1 (Pin_1), U3.37 (3V3_EN)
- new net: R2.1, U6.18 (B0)
- new net: J5.1 (Pin_1), R2.2
- new net: R1.2, U4.1 (A->B), U4.8 (A6), U4.9 (A7), U5.1 (A->B), U5.8 (A6), U5.9 (A7), U6.1 (A->B), U7.1 (A->B), U7.8 (A6), U7.9 (A7)
- new net: J5.2 (Pin_2), R3.2
- new net: J5.3 (Pin_3), R4.2
- new net: R3.1, U6.14 (B4)
- new net: D1.1 (K), U3.39 (VSYS)
- new net: R4.1, U7.18 (B0)
- new net 2MHZ: U10.54 (2MHZ), U11.54 (2MHZ)
- new net 3V3: C2.1, C3.1, C5.1, C6.1, C7.1, U8.2 (VO), U9.26 (VCCIO), U9.38 (VCCIO), U9.5 (VCCINT), U9.51 (VCCIO), U9.57 (VCCINT), U9.88 (VCCIO), U9.98 (VCCINT)
- new net 500KHZ: U10.43 (500KHZ), U11.43 (500KHZ)
- new net 6850CS: U10.42 (6850CS), U11.42 (6850CS)
- new net 8MHZ: U10.34 (8MHZ), U11.34 (8MHZ), U9.22 (I/O/GCK1)
- new net A10: U10.65 (A10), U11.65 (A10), U9.78 (P78)
- new net A11: U10.66 (A11), U11.66 (A11), U9.77 (P77)
- new net A12: U10.67 (A12), U11.67 (A12), U9.76 (P76)
- new net A13: U10.68 (A13), U11.68 (A13), U9.74 (P74)
- new net A14: U10.2 (A14), U11.2 (A14), U9.49 (P49)
- new net A15: U10.3 (A15), U11.3 (A15), U9.46 (P46)
- new net A16: U10.4 (A16), U11.4 (A16), U9.43 (P43)
- new net A17: U10.5 (A17), U11.5 (A17), U9.42 (P42)
- new net A18: U10.6 (A18), U11.6 (A18), U9.41 (P41)
- new net A19: U10.7 (A19), U11.7 (A19), U9.40 (P40)
- new net A20: U10.8 (A20), U11.8 (A20), U9.39 (P39)
- new net A21: U10.9 (A21), U11.9 (A21), U9.37 (P37)
- new net A22: U10.10 (A22), U11.10 (A22), U9.36 (P36)
- new net A23: U10.11 (A23), U11.11 (A23), U9.35 (P35)
- new net A6: U10.61 (A6), U11.61 (A6), U9.82 (P82)
- new net A7: U10.62 (A7), U11.62 (A7), U9.81 (P81)
- new net A8: U10.63 (A8), U11.63 (A8), U9.80 (P80)
- new net A9: U10.64 (A9), U11.64 (A9), U9.79 (P79)
- new net AS: U10.12 (~{AS}), U11.12 (~{AS}), U9.12 (P12)
- new net BERR: U10.30 (~{BERR}), U11.30 (~{BERR})
- new net BGI: U10.27 (~{BGI}), U11.27 (~{BGI})
- new net BGK: U10.41 (~{BGACK}), U11.41 (~{BGACK})
- new net BGO: U10.45 (~{BGO}), U11.45 (~{BGO})
- new net BLANK: U11.36 (~{BLANK}), U9.9 (P9)
- new net BLANK_OUT: U10.36 (~{BLANK}), U9.10 (P10)
- new net BR: U10.40 (~{BR}), U11.40 (~{BR})
- new net D0_C: J6.3 (Pin_3), U9.55 (P55)
- new net D10_C: J6.13 (Pin_13), U9.67 (P67)
- new net D11_C: J6.14 (Pin_14), U9.68 (P68)
- new net D12_C: J6.15 (Pin_15), U9.70 (P70)
- new net D13_C: J6.16 (Pin_16), U9.71 (P71)
- new net D14_C: J6.17 (Pin_17), U9.72 (P72)
- new net D15_C: J6.18 (Pin_18), U9.73 (P73)
- new net D1_C: J6.4 (Pin_4), U9.56 (P56)
- new net D2_C: J6.5 (Pin_5), U9.58 (P58)
- new net D3_C: J6.6 (Pin_6), U9.59 (P59)
- new net D4_C: J6.7 (Pin_7), U9.60 (P60)
- new net D5_C: J6.8 (Pin_8), U9.61 (P61)
- new net D6_C: J6.9 (Pin_9), U9.63 (P63)
- new net D7_C: J6.10 (Pin_10), U9.64 (P64)
- new net D8_C: J6.11 (Pin_11), U9.65 (P65)
- new net D9_C: J6.12 (Pin_12), U9.66 (P66)
- new net DEV: U10.25 (~{DEV}), U11.25 (~{DEV})
- new net DMA: U10.24 (~{DMA}), U11.24 (~{DMA})
- new net DTACK: U10.31 (~{DTACK}), U11.31 (~{DTACK}), U9.15 (P15)
- new net FC0: U10.15 (FC0), U11.15 (FC0)
- new net FC1: U10.14 (FC1), U11.14 (FC1)
- new net FC2: U10.13 (FC2), U11.13 (FC2)
- new net FCS: U10.26 (~{FCS}), U11.26 (~{FCS})
- new net HSYNC: U11.37 (HSYNC), U9.6 (P6)
- new net HSYNC_OUT: U10.37 (HSYNC), U9.8 (P8)
- new net IACK: U10.50 (~{IACK}), U11.50 (~{IACK})
- new net IPL1: U10.32 (~{IPL1}), U11.32 (~{IPL1})
- new net IPL2: U10.33 (~{IPL2}), U11.33 (~{IPL2})
- new net LDS: U10.46 (~{LDS}), U11.46 (~{LDS}), U9.13 (P13)
- new net MFPCS: U10.51 (~{MFPCS}), U11.51 (~{MFPCS})
- new net MFPINT: U10.44 (~{MFPINT}), U11.44 (~{MFPINT})
- new net OSC: U9.23 (I/O/GCK2), X1.8 (OUT)
- new net PICOB0: J2.10 (Pin_10), U3.11 (GPIO8), U6.6 (A4)
- new net PICOB1: J2.11 (Pin_11), U3.12 (GPIO9), U6.7 (A5)
- new net PICOB2: J2.12 (Pin_12), U3.14 (GPIO10), U6.8 (A6)
- new net PICOB3: J2.13 (Pin_13), U3.15 (GPIO11), U6.9 (A7)
- new net PICOG0: J2.6 (Pin_6), U3.6 (GPIO4), U6.2 (A0)
- new net PICOG1: J2.7 (Pin_7), U3.7 (GPIO5), U6.3 (A1)
- new net PICOG2: J2.8 (Pin_8), U3.9 (GPIO6), U6.4 (A2)
- new net PICOG3: J2.9 (Pin_9), U3.10 (GPIO7), U6.5 (A3)
- new net PICOHSYNC: J1.18 (Pin_18), J2.15 (Pin_15), U3.17 (GPIO13)
- new net PICOHSYNC_C: J7.18 (Pin_18), U9.97 (P97)
- new net PICOR0: J2.2 (Pin_2), U3.1 (GPIO0), U7.2 (A0)
- new net PICOR1: J2.3 (Pin_3), U3.2 (GPIO1), U7.3 (A1)
- new net PICOR2: J2.4 (Pin_4), U3.4 (GPIO2), U7.4 (A2)
- new net PICOR3: J2.5 (Pin_5), U3.5 (GPIO3), U7.5 (A3)
- new net PICOVSYNC: J1.17 (Pin_17), J2.14 (Pin_14), U3.16 (GPIO12)
- new net PICOVSYNC_C: J7.17 (Pin_17), U9.96 (P96)
- new net PICO_A0: J1.5 (Pin_5), U3.31 (GPIO26_ADC0)
- new net PICO_A0_C: J7.5 (Pin_5), U9.30 (P30)
- new net PICO_A1: J1.4 (Pin_4), U3.32 (GPIO27_ADC1)
- new net PICO_A1_C: J7.4 (Pin_4), U9.29 (P29)
- new net PICO_A2: J1.3 (Pin_3), U3.34 (GPIO28_ADC2)
- new net PICO_A2_C: J7.3 (Pin_3), U9.28 (P28)
- new net PICO_CLK: J1.6 (Pin_6), U3.29 (GPIO22)
- new net PICO_CLK_C: J7.6 (Pin_6), U9.32 (P32)
- new net PICO_D0: J1.14 (Pin_14), U3.19 (GPIO14)
- new net PICO_D0_C: J7.14 (Pin_14), U9.93 (P93)
- new net PICO_D1: J1.13 (Pin_13), U3.20 (GPIO15)
- new net PICO_D1_C: J7.13 (Pin_13), U9.92 (P92)
- new net PICO_D2: J1.12 (Pin_12), U3.21 (GPIO16)
- new net PICO_D2_C: J7.12 (Pin_12), U9.91 (P91)
- new net PICO_D3: J1.11 (Pin_11), U3.22 (GPIO17)
- new net PICO_D3_C: J7.11 (Pin_11), U9.90 (P90)
- new net PICO_D4: J1.10 (Pin_10), U3.24 (GPIO18)
- new net PICO_D4_C: J7.10 (Pin_10), U9.89 (P89)
- new net PICO_D5: J1.9 (Pin_9), U3.25 (GPIO19)
- new net PICO_D5_C: J7.9 (Pin_9), U9.87 (P87)
- new net PICO_D6: J1.8 (Pin_8), U3.26 (GPIO20)
- new net PICO_D6_C: J7.8 (Pin_8), U9.34 (P34)
- new net PICO_D7: J1.7 (Pin_7), U3.27 (GPIO21)
- new net PICO_D7_C: J7.7 (Pin_7), U9.33 (P33)
- new net RAM: U10.23 (~{RAM}), U11.23 (~{RAM})
- new net RDY: U10.28 (RDY), U11.28 (RDY)
- new net RESET: U10.22 (~{RESET}), U11.22 (~{RESET}), U9.99 (I/O/GSR)
- new net ROM0: U10.21 (~{ROM0}), U11.21 (~{ROM0})
- new net ROM1: U10.20 (~{ROM1}), U11.20 (~{ROM1})
- new net ROM2: U10.19 (~{ROM2}), U11.19 (~{ROM2})
- new net ROM3: U10.18 (~{ROM3}), U11.18 (~{ROM3})
- new net ROM4: U10.17 (~{ROM4}), U11.17 (~{ROM4})
- new net SNDCS: U10.53 (~{SNDCS}), U11.53 (~{SNDCS})
- new net TEST: U10.52 (TEST), U11.52 (TEST)
- new net UDS: U10.47 (~{UDS}), U11.47 (~{UDS}), U9.14 (P14)
- new net VMA: U10.16 (~{VMA}), U11.16 (~{VMA})
- new net VPA: U10.29 (~{VPA}), U11.29 (~{VPA})
- new net VSYNC: U11.38 (VSYNC), U9.4 (I/O/GTS2)
- new net VSYNC_OUT: U10.38 (VSYNC), U9.7 (P7)
- new net ~{PICOEN_C}: J7.16 (Pin_16), U9.95 (P95)
- new net ~{PICOEN_P}: J1.16 (Pin_16), U6.19 (CE), U7.19 (CE)
- new net ~{SHIFTEREN_C}: J7.15 (Pin_15), U9.94 (P94)
- new net ~{SHIFTEREN_P}: J1.15 (Pin_15), U4.19 (CE), U5.19 (CE)
- no-connect marks 0 -> 18
Other:
- removed sheet Glue Board
- note added: "Not all pins set! Check RGB 0-3 ordering!"
- note added: "Pins not set! Look at what we use on prototype"
- note added: "STE VIDEO BIT OUT"

Commit message: Adding libs and initial draft of schematic complete
Parts:
- added J8: Conn_01x06_Male, symbol Connector:Conn_01x06_Male
- added R5: 1k, symbol Device:R
- added R6: 68R, symbol Device:R
Connections:
- net 3V3: now also R5.1
- net 5V: no longer C1.1, C4.1, U10.1 (VCC), U11.1 (VCC), U8.3 (VI), X1.14 (Vcc)
- net GND: no longer C1.2, C2.2, C3.2, C4.2, C5.2, C6.2, C7.2, J6.1 (Pin_1), J6.19 (Pin_19), J6.2 (Pin_2), J6.20 (Pin_20), J7.1 (Pin_1), J7.19 (Pin_19), J7.2 (Pin_2), J7.20 (Pin_20), U10.35 (GND), U11.35 (GND), U8.1 (GND), U9.100 (GND), U9.21 (GND), U9.31 (GND), U9.44 (GND), U9.62 (GND), U9.69 (GND), U9.75 (GND), U9.84 (GND), X1.7 (GND)
- net OSC: now also R6.2; no longer X1.8 (OUT)
- net at R1.2, U4.1 (A->B), U4.8 (A6)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: now also U5.6 (A4), U5.7 (A5), U7.6 (A4), U7.7 (A5)
- net TDI: now reaches U9.45 (TDI)
- net TDI: now also J8.5 (Pin_5)
- net TMS: now reaches U9.47 (TMS)
- net TMS: now also J8.6 (Pin_6)
- net TCK: now reaches U9.48 (TCK)
- net TCK: now also J8.3 (Pin_3)
- net TDO: now reaches U9.83 (TDO)
- net TDO: now also J8.4 (Pin_4)
- new net 3V3_SENSE: J8.1 (Pin_1), R5.2
- new net 5V_C: C1.1, C4.1, U10.1 (VCC), U11.1 (VCC), U8.3 (VI), X1.14 (Vcc)
- new net GND_C: C1.2, C2.2, C3.2, C4.2, C5.2, C6.2, C7.2, J6.1 (Pin_1), J6.19 (Pin_19), J6.2 (Pin_2), J6.20 (Pin_20), J7.1 (Pin_1), J7.19 (Pin_19), J7.2 (Pin_2), J7.20 (Pin_20), J8.2 (Pin_2), U10.35 (GND), U11.35 (GND), U8.1 (GND), U9.100 (GND), U9.21 (GND), U9.31 (GND), U9.44 (GND), U9.62 (GND), U9.69 (GND), U9.75 (GND), U9.84 (GND), X1.7 (GND)
- new net OSC_OUT: R6.1, X1.8 (OUT)
- no-connect marks 18 -> 30

Commit message: Experimenting with board layout
Parts:
- removed J1, J3, J6, J7: Conn_01x20, symbol Connector_Generic:Conn_01x20
- added J2, J3, J6, J7: F3311A7H121020E200, F3311A7H121020E200:AMPHENOL_F3311A7H121020E200, symbol F3311A7H121020E200:F3311A7H121020E200
- C1, C2, C3, C4, C5, C6, C7: footprint (none) -> Capacitor_SMD:C_0805_2012Metric_Pad1.18x1.45mm_HandSolder
- D1: footprint (none) -> Diode_SMD:D_0805_2012Metric_Pad1.15x1.40mm_HandSolder
- J1: renamed from J2; footprint (none) -> Connector_PinHeader_2.54mm:PinHeader_1x16_P2.54mm_Horizontal
- J4: footprint (none) -> Connector_PinHeader_2.54mm:PinHeader_1x02_P2.54mm_Vertical
- J5: footprint (none) -> Connector_PinHeader_2.54mm:PinHeader_1x03_P2.54mm_Horizontal
- J8: footprint (none) -> Connector_PinHeader_2.54mm:PinHeader_1x06_P2.54mm_Horizontal
- R1, R2, R3, R4, R5, R6: footprint (none) -> Resistor_SMD:R_0805_2012Metric_Pad1.20x1.40mm_HandSolder
- U3: footprint RPi_Pico:RPi_Pico_SMD_TH -> MCU_RaspberryPi_and_Boards:RPi_Pico_SMD_TH
- U4, U5, U6, U7: footprint (none) -> Package_SO:TSSOP-20_4.4x6.5mm_P0.65mm
- U8: footprint (none) -> Package_TO_SOT_SMD:SOT-23
Connections:
- net D0: now also J3.3
- net D0_C: now also J6.3
- net D1: now also J3.4
- net D10: now also J3.13
- net D10_C: now also J6.13
- net D11: now also J3.14
- net D11_C: now also J6.14
- net D12: now also J3.15
- net D12_C: now also J6.15
- net D13: now also J3.16
- net D13_C: now also J6.16
- net D14: now also J3.17
- net D14_C: now also J6.17
- net D15: now also J3.18
- net D15_C: now also J6.18
- net D1_C: now also J6.4
- net D2: now also J3.5
- net D2_C: now also J6.5
- net D3: now also J3.6
- net D3_C: now also J6.6
- net D4: now also J3.7
- net D4_C: now also J6.7
- net D5: now also J3.8
- net D5_C: now also J6.8
- net D6: now also J3.9
- net D6_C: now also J6.9
- net D7: now also J3.10
- net D7_C: now also J6.10
- net D8: now also J3.11
- net D8_C: now also J6.11
- net D9: now also J3.12
- net D9_C: now also J6.12
- net GND: now also J2.1, J2.19, J2.2, J2.20, J3.1, J3.19, J3.2, J3.20
- net GND_C: now also J6.1, J6.19, J6.2, J6.20, J7.1, J7.19, J7.2, J7.20
- net MONO: now also U5.2 (A0); no longer U5.5 (A3)
- net MONO_OUT: now also U5.18 (B0); no longer U5.15 (B3)
- net PICOHSYNC: now also J2.18
- net PICOHSYNC_C: now also J7.18
- net PICOVSYNC: now also J2.17
- net PICOVSYNC_C: now also J7.17
- net PICO_A0: now also J2.5
- net PICO_A0_C: now also J7.5
- net PICO_A1: now also J2.4
- net PICO_A1_C: now also J7.4
- net PICO_A2: now also J2.3
- net PICO_A2_C: now also J7.3
- net PICO_CLK: now also J2.6
- net PICO_CLK_C: now also J7.6
- net PICO_D0: now also J2.14
- net PICO_D0_C: now also J7.14
- net PICO_D1: now also J2.13
- net PICO_D1_C: now also J7.13
- net PICO_D2: now also J2.12
- net PICO_D2_C: now also J7.12
- net PICO_D3: now also J2.11
- net PICO_D3_C: now also J7.11
- net PICO_D4: now also J2.10
- net PICO_D4_C: now also J7.10
- net PICO_D5: now also J2.9
- net PICO_D5_C: now also J7.9
- net PICO_D6: now also J2.8
- net PICO_D6_C: now also J7.8
- net PICO_D7: now also J2.7
- net PICO_D7_C: now also J7.7
- net R0: now also U5.3 (A1); no longer U5.2 (A0)
- net R1: now also U5.4 (A2); no longer U5.3 (A1)
- net R2: now also U5.5 (A3); no longer U5.4 (A2)
- net R_OUT0: now also U5.17 (B1); no longer U5.18 (B0)
- net R_OUT1: now also U5.16 (B2); no longer U5.17 (B1)
- net R_OUT2: now also U5.15 (B3); no longer U5.16 (B2)
- net ~{PICOEN_C}: now also J7.16
- net ~{PICOEN_P}: now also J2.16
- net ~{SHIFTEREN_C}: now also J7.15
- net ~{SHIFTEREN_P}: now also J2.15

Commit message: More layout experimentation
Connections:
- net B_OUT0: now also U6.16 (B2); no longer U6.13 (B5)
- net B_OUT1: now also U6.17 (B1); no longer U6.12 (B6)
- net B_OUT2: now also U6.18 (B0); no longer U6.11 (B7)
- net G_OUT0: now also U7.14 (B4); no longer U6.17 (B1)
- net G_OUT1: now also U7.15 (B3); no longer U6.16 (B2)
- net G_OUT2: now also U7.16 (B2); no longer U6.15 (B3)
- net PICOB0: now also U6.7 (A5); no longer U6.6 (A4)
- net PICOB1: now also U6.4 (A2); no longer U6.7 (A5)
- net PICOB2: now also U6.3 (A1); no longer U6.8 (A6)
- net PICOB3: now also U6.2 (A0); no longer U6.9 (A7)
- net PICOG0: now also U6.8 (A6); no longer U6.2 (A0)
- net PICOG1: now also U7.6 (A4); no longer U6.3 (A1)
- net PICOG2: now also U7.5 (A3); no longer U6.4 (A2)
- net PICOG3: now also U7.4 (A2); no longer U6.5 (A3)
- net PICOR0: now also U6.9 (A7); no longer U7.2 (A0)
- net PICOR1: now also U7.9 (A7); no longer U7.3 (A1)
- net PICOR2: now also U7.8 (A6); no longer U7.4 (A2)
- net PICOR3: now also U7.7 (A5); no longer U7.5 (A3)
- net R_OUT0: now also U7.11 (B7); no longer U7.17 (B1)
- net R_OUT1: now also U7.12 (B6); no longer U7.16 (B2)
- net R_OUT2: now also U7.13 (B5); no longer U7.15 (B3)
- net ~{PICOEN_P}: no longer U7.19 (CE)
- net at R2.1: now also U6.11 (B7); no longer U6.18 (B0)
- net R_STE: now reaches J5.1 (Pin_1), R2.2
- net at R1.2, U4.1 (A->B), U4.8 (A6)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: no longer U7.6 (A4), U7.7 (A5), U7.8 (A6), U7.9 (A7)
- net G_STE: now reaches J5.2 (Pin_2), R3.2
- net B_STE: now reaches J5.3 (Pin_3), R4.2
- net at R3.1: now also U6.12 (B6); no longer U6.14 (B4)
- net at R4.1: now also U6.13 (B5); no longer U7.18 (B0)
Other:
- moved on the sheet: J5, R2, R3, R4

Commit message: Preliminary routeing of shifter board nearly complete
Parts:
- removed C1, C2: 1u, Capacitor_SMD:C_0805_2012Metric_Pad1.18x1.45mm_HandSolder, symbol Device:C
- removed J1: Conn_01x16_Female, Connector_PinHeader_2.54mm:PinHeader_1x16_P2.54mm_Horizontal, symbol Connector:Conn_01x16_Female
- removed U8: LM1117-3.3, Package_TO_SOT_SMD:SOT-23, symbol Regulator_Linear:LM1117-3.3
- added R2, R3: 10k, Resistor_SMD:R_0805_2012Metric_Pad1.20x1.40mm_HandSolder, symbol Device:R
- U9: renamed from U10; footprint Package_LCC:PLCC-68_THT-Socket -> PLCC_plugs:PLCC68_male_pins
- renumbered C3 to C1, C4 to C2, C5 to C3, C6 to C4, C7 to C5, J2 to J1, J3 to J2, J4 to J3, J5 to J4, J6 to J5, J7 to J6, J8 to J7, R2 to R4, R3 to R5, R4 to R6, R5 to R7, R6 to R8, U11 to U10, U9 to U8
Connections:
- net 3V3: now also U3.36 (3V3)
- net 5V: now also R3.2
- net B_OUT0: now also U6.11 (B7); no longer U6.16 (B2)
- net B_OUT1: now also U6.12 (B6); no longer U6.17 (B1)
- net B_OUT2: now also U6.13 (B5); no longer U6.18 (B0)
- net GND: now also R2.1; no longer J3.2 (Pin_2), U3.13 (GND), U3.18 (GND), U3.23 (GND), U3.28 (GND), U3.3 (GND), U3.33 (AGND), U3.38 (GND), U3.8 (GND)
- net GND_C: now also J3.2 (Pin_2), U3.13 (GND), U3.18 (GND), U3.23 (GND), U3.28 (GND), U3.3 (GND), U3.33 (AGND), U3.38 (GND), U3.8 (GND)
- net PICOB0: now also J1.16, J6.11, U6.4 (A2); no longer U6.7 (A5)
- net PICOB1: now also J1.13, J6.12, U6.9 (A7); no longer U6.4 (A2)
- net PICOB2: now also J1.14, J6.13, U6.8 (A6); no longer U6.3 (A1)
- net PICOB3: now also J1.15, J6.14, U6.7 (A5); no longer U6.2 (A0)
- net PICOG0: now also J1.17, J6.7, U6.3 (A1); no longer U6.8 (A6)
- net PICOG1: now also J1.10, J6.8
- net PICOG2: now also J1.11, J6.9
- net PICOG3: now also J1.12, J6.10
- net PICOHSYNC: no longer J1.18
- net PICOHSYNC_C: no longer J6.18
- net PICOR0: now also J1.18, J6.3, U6.2 (A0); no longer U6.9 (A7)
- net PICOR1: now also J1.7, J6.4
- net PICOR2: now also J1.8, J6.5
- net PICOR3: now also J1.9, J6.6
- net PICOVSYNC: no longer J1.17
- net PICOVSYNC_C: no longer J6.17
- net PICO_A0: no longer J1.5
- net PICO_A0_C: no longer J6.5
- net PICO_A1: no longer J1.4
- net PICO_A1_C: no longer J6.4
- net PICO_A2: no longer J1.3
- net PICO_A2_C: no longer J6.3
- net PICO_CLK: no longer J1.6
- net PICO_CLK_C: no longer J6.6
- net PICO_D0: no longer J1.14
- net PICO_D0_C: no longer J6.14
- net PICO_D1: no longer J1.13
- net PICO_D1_C: no longer J6.13
- net PICO_D2: no longer J1.12
- net PICO_D2_C: no longer J6.12
- net PICO_D3: no longer J1.11
- net PICO_D3_C: no longer J6.11
- net PICO_D4: no longer J1.10
- net PICO_D4_C: no longer J6.10
- net PICO_D5: no longer J1.9
- net PICO_D5_C: no longer J6.9
- net PICO_D6: no longer J1.8
- net PICO_D6_C: no longer J6.8
- net PICO_D7: no longer J1.7
- net PICO_D7_C: no longer J6.7
- net ~{PICOEN_C}: now also J6.18; no longer J6.16
- net ~{PICOEN_P}: now also J1.3, U7.19 (CE), R3.1; no longer J1.16
- net ~{SHIFTEREN_C}: now also J6.17; no longer J6.15
- net ~{SHIFTEREN_P}: now also J1.4, R2.2; no longer J1.15
- net at R4.1: now also U6.18 (B0); no longer U6.11 (B7)
- net 5VPULL: now reaches R1.2, U4.1 (A->B), U4.8 (A6), U4.9 (A7), U5.1 (A->B), U5.6 (A4), U5.7 (A5), U5.8 (A6), U5.9 (A7), U6.1 (A->B), U7.1 (A->B)
- net 5VPULL: now also U6.5 (A3), U6.6 (A4), U7.2 (A0), U7.3 (A1)
- net at R5.1: now also U6.17 (B1); no longer U6.12 (B6)
- net at R6.1: now also U6.16 (B2); no longer U6.13 (B5)
- no-connect marks 30 -> 29
Other:
- moved on the sheet: J4, R1, R4, R5, R6
