File: kicad/video_rider_st.kicad_sch (KiCad schematic)
At the start: 32 parts, among them J1 F3311A7H121020E200, J2 F3311A7H121020E200, J3 Conn_01x02_Male, J4 Conn_01x03_Male, J5 F3311A7H121020E200, J6 F3311A7H121020E200, J7 Conn_01x06_Male, U1 ST_SHIFTER_PHY, U10 ST_GLUE_SOCKET, U2 ST_SHIFTER_SOCKET, U3 Pico, U4 74HC245, U5 74HC245, U6 74HC245, U7 74HC245, U8 XC95144XL-TQ100, U9 ST_GLUE_PHY, X1 CXO_DIP14

Commit message: Adding support for other oscillators
Parts:
- removed X1: CXO_DIP14, Oscillator:Oscillator_DIP-14, symbol Oscillator:CXO_DIP14
- added C6: 1u, Capacitor_SMD:C_0805_2012Metric_Pad1.18x1.45mm_HandSolder, symbol Device:C
- added TP1, TP2, TP3, TP4: TestPoint, TestPoint:TestPoint_THTPad_1.5x1.5mm_Drill0.7mm, symbol Connector:TestPoint
- added X1: CXO_DIP14_DIP8_DUAL, CXO_Dual_DIP:CXO_Dual_DIP, symbol cxo_dip14_dip8_dual:CXO_DIP14_DIP8_DUAL
Connections:
- net 3V3: now also J6.15, J6.16
- net 5V_C: now also C6.1, X1.14 (Vcc)
- net BLANK_OUT: now also U8.6 (P6); no longer U8.4 (I/O/GTS2)
- net D0_C: now also U8.94 (P94); no longer U8.76 (P76)
- net D10_C: now also U8.81 (P81); no longer U8.89 (P89)
- net D11_C: now also U8.80 (P80); no longer U8.90 (P90)
- net D12_C: now also U8.79 (P79); no longer U8.91 (P91)
- net D13_C: now also U8.78 (P78); no longer U8.92 (P92)
- net D14_C: now also U8.77 (P77); no longer U8.93 (P93)
- net D15_C: now also U8.76 (P76); no longer U8.94 (P94)
- net D1_C: now also U8.93 (P93); no longer U8.77 (P77)
- net D2_C: now also U8.92 (P92); no longer U8.78 (P78)
- net D3_C: now also U8.91 (P91); no longer U8.79 (P79)
- net D4_C: now also U8.90 (P90); no longer U8.80 (P80)
- net D5_C: now also U8.89 (P89); no longer U8.81 (P81)
- net D6_C: now also U8.87 (P87); no longer U8.82 (P82)
- net D7_C: now also U8.86 (P86); no longer U8.85 (P85)
- net D8_C: now also U8.85 (P85); no longer U8.86 (P86)
- net D9_C: now also U8.82 (P82); no longer U8.87 (P87)
- net GND_C: now also C6.2, X1.4 (GND), X1.7 (GND)
- net HSYNC_OUT: now also U8.7 (P7); no longer U8.6 (P6)
- net OSC_OUT: now also X1.11 (OUT), X1.8 (OUT)
- net PICO_A0: now also U8.59 (P59); no longer U8.58 (P58)
- net PICO_A1: now also U8.60 (P60); no longer U8.56 (P56)
- net PICO_A2: now also U8.61 (P61); no longer U8.55 (P55)
- net PICO_CLK: now also U8.58 (P58); no longer U8.59 (P59)
- net PICO_D0: now also U8.64 (P64); no longer U8.67 (P67)
- net PICO_D1: now also U8.63 (P63); no longer U8.68 (P68)
- net PICO_D2: now also U8.50 (P50); no longer U8.71 (P71)
- net PICO_D3: now also U8.52 (P52); no longer U8.70 (P70)
- net PICO_D4: now also U8.53 (P53); no longer U8.64 (P64)
- net PICO_D5: now also U8.54 (P54); no longer U8.63 (P63)
- net PICO_D6: now also U8.55 (P55); no longer U8.61 (P61)
- net PICO_D7: now also U8.56 (P56); no longer U8.60 (P60)
- net VSYNC_OUT: now also U8.8 (P8); no longer U8.7 (P7)
- net TP1: now reaches U8.1 (I/O/GTS3)
- net TP1: now also TP1.1
- net TP2: now reaches U8.2 (I/O/GTS4)
- net TP2: now also TP2.1
- net TP3: now reaches U8.3 (I/O/GTS1)
- net TP3: now also TP3.1
- new net TP4: TP4.1, U8.4 (I/O/GTS2)
- no-connect marks 29 -> 27
Other:
- moved on the sheet: C2, R8
