File: kicad_shifterboard/vr_shifterboard.kicad_pcb (KiCad board)
At the start: 2 copper layers, 57.3 x 34.1 mm, 20 parts, among them J1 F3311A7H121020E200, J2 F3311A7H121020E200, J4 Conn_01x03_Male, U1 ST_SHIFTER_PHY, U2 ST_SHIFTER_SOCKET, U4 74HC245, U5 74HC245, U6 74HC245, U7 74HC245

Commit message: Preparing gerbers again
Connections:
- J1 pad SH1: (no net) -> /GND
- J1 pad SH2: (no net) -> /GND
- J2 pad SH1: (no net) -> /GND
- J2 pad SH2: (no net) -> /GND
Other:
- board text added: "Shifter board v0.2 Copyright D Henderson 2025"
- board text removed: "Copyright D Henderson 2025"
Changed lines of the file:
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@@
       (drillshape 0)
       (scaleselection 1)
-      (outputdirectory "gerbers")
+      (outputdirectory "shifterboard")
     )
   )
@@
       (net 2 "/GND") (pinfunction "20") (pintype "passive"))
     (pad "SH1" smd rect locked (at -5.75 0.925 90) (size 0.4 0.8) (layers "F.Cu" "F.Paste" "F.Mask")
-      (solder_mask_margin 0.102))
+      (net 2 "/GND") (solder_mask_margin 0.102))
     (pad "SH2" smd rect locked (at 5.75 0.925 90) (size 0.4 0.8) (layers "F.Cu" "F.Paste" "F.Mask")
-      (solder_mask_margin 0.102))
+      (net 2 "/GND") (solder_mask_margin 0.102))
   )
   (footprint "Package_SO:TSSOP-20_4.4x6.5mm_P0.65mm" (layer "F.Cu")
@@
       (net 2 "/GND") (pinfunction "20") (pintype "passive"))
     (pad "SH1" smd rect locked (at -5.75 0.925 90) (size 0.4 0.8) (layers "F.Cu" "F.Paste" "F.Mask")
-      (solder_mask_margin 0.102))
+      (net 2 "/GND") (solder_mask_margin 0.102))
     (pad "SH2" smd rect locked (at 5.75 0.925 90) (size 0.4 0.8) (layers "F.Cu" "F.Paste" "F.Mask")
-      (solder_mask_margin 0.102))
+      (net 2 "/GND") (solder_mask_margin 0.102))
   )
   (footprint "Capacitor_SMD:C_0805_2012Metric_Pad1.18x1.45mm_HandSolder" (layer "B.Cu")
@@
     (effects (font (size 2 1.1) (thickness 0.275) italic) (justify left))
   )
-  (gr_text "Copyright D Henderson 2025" (at 87.9 62.8) (layer "F.SilkS")
+  (gr_text "Shifter board v0.2\nCopyright D Henderson 2025" (at 87.9 62.8) (layer "F.SilkS")
     (effects (font (size 0.7 0.7) (thickness 0.1)) (justify left))
   )
