File: kicad_glueboard/vr_glueboard.kicad_pcb (KiCad board)
At the start: 2 copper layers, 99 x 57.6 mm, 23 parts, among them J3 Conn_01x02_Male, J5 F3311A7H121020E200, J6 F3311A7H121020E200, J7 Conn_01x06_Male, U10 ST_GLUE_SOCKET, U3 Pico, U8 XC95144XL-TQ100, U9 ST_GLUE_PHY, X1 CXO_DIP14_DIP8_DUAL, X2 IQXO-70

Commit message: Preparing gerbers again
Connections:
- J5 pad SH1: /GND_C -> (no net)
- J5 pad SH2: /GND_C -> (no net)
- J6 pad SH1: /GND_C -> (no net)
- J6 pad SH2: /GND_C -> (no net)
Changed lines of the file:
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@@
       (drillshape 0)
       (scaleselection 1)
-      (outputdirectory "gerbers")
+      (outputdirectory "glueboard")
     )
   )
@@
       (net 2 "/GND_C") (pinfunction "20") (pintype "passive"))
     (pad "SH1" smd rect locked (at -5.75 0.925 180) (size 0.4 0.8) (layers "F.Cu" "F.Paste" "F.Mask")
-      (net 2 "/GND_C") (solder_mask_margin 0.102))
+      (solder_mask_margin 0.102))
     (pad "SH2" smd rect locked (at 5.75 0.925 180) (size 0.4 0.8) (layers "F.Cu" "F.Paste" "F.Mask")
-      (net 2 "/GND_C") (solder_mask_margin 0.102))
+      (solder_mask_margin 0.102))
   )
   (footprint "Connector_PinHeader_2.54mm:PinHeader_1x06_P2.54mm_Vertical" (layer "F.Cu")
@@
       (net 2 "/GND_C") (pinfunction "20") (pintype "passive"))
     (pad "SH1" smd rect locked (at -5.75 0.925 180) (size 0.4 0.8) (layers "F.Cu" "F.Paste" "F.Mask")
-      (net 2 "/GND_C") (solder_mask_margin 0.102))
+      (solder_mask_margin 0.102))
     (pad "SH2" smd rect locked (at 5.75 0.925 180) (size 0.4 0.8) (layers "F.Cu" "F.Paste" "F.Mask")
-      (net 2 "/GND_C") (solder_mask_margin 0.102))
+      (solder_mask_margin 0.102))
   )
   (footprint "Capacitor_SMD:C_0805_2012Metric_Pad1.18x1.45mm_HandSolder" (layer "B.Cu")

Commit message: A few mods to to the glueboard to ensure trace/edge cut separation and just some tiding up. Changed pico data pin order to get a better ground.
Connections:
- J5 pad SH1: (no net) -> /GND_C
- J5 pad SH2: (no net) -> /GND_C
- J6 pad SH1: (no net) -> /GND_C
- J6 pad SH2: (no net) -> /GND_C
- U8 pad 50: /PICO_D2 -> /PICO_D3
- U8 pad 52: /PICO_D3 -> /PICO_D4
- U8 pad 53: /PICO_D4 -> /PICO_D2
Routing:
- net /PICOG2_C: track 37.9 -> 42.2 mm
- net /PICO_D2: track 43.2 -> 46.3 mm
- net /PICOG3_C: track 40.0 -> 42.8 mm
- net /PICO_D3: track 41.4 -> 42.5 mm
- net /PICOB1_C: track 45.4 -> 44.5 mm
- net /PICO_D5: track 33.6 -> 34.3 mm
- net /PICOB3_C: track 47.3 -> 46.6 mm
- net /PICOR2_C: track 24.5 -> 25.2 mm
- net /PICOVSYNC: track 58.9 -> 58.3 mm
- net /PICOHSYNC: track 61.5 -> 60.9 mm
