File: kicad_glueboard/vr_glueboard.kicad_sch (KiCad schematic)
At the start: 23 parts, among them J3 Conn_01x02_Male, J5 F3311A7H121020E200, J6 F3311A7H121020E200, J7 Conn_01x06_Male, U10 ST_GLUE_SOCKET, U3 Pico, U8 XC95144XL-TQ100, U9 ST_GLUE_PHY, X1 CXO_DIP14_DIP8_DUAL, X2 IQXO-70

Commit message: A few mods to to the glueboard to ensure trace/edge cut separation and just some tiding up. Changed pico data pin order to get a better ground.
Connections:
- net PICO_D2: now also U8.53 (P53); no longer U8.50 (P50)
- net PICO_D3: now also U8.50 (P50); no longer U8.52 (P52)
- net PICO_D4: now also U8.52 (P52); no longer U8.53 (P53)
Changed lines of the file:
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@@
     (effects (font (size 1.27 1.27)) (justify right bottom))
   )
-  (label "PICO_D2" (at 245.11 154.305 180)
+  (label "PICO_D2" (at 245.11 159.385 180)
     (effects (font (size 1.27 1.27)) (justify right bottom))
   )
@@
     (effects (font (size 1.27 1.27)) (justify right bottom))
   )
-  (label "PICO_D4" (at 245.11 159.385 180)
+  (label "PICO_D4" (at 245.11 156.845 180)
     (effects (font (size 1.27 1.27)) (justify right bottom))
   )
@@
     (effects (font (size 1.27 1.27)) (justify right bottom))
   )
-  (label "PICO_D3" (at 245.11 156.845 180)
-    (effects (font (size 1.27 1.27)) (justify right bottom))
-  )
+  (label "PICO_D3" (at 245.11 154.305 180)
+    (effects (font (size 1.27 1.27)) (justify right bottom))
+  )
